Commit message: camera urdf stuff

File: resources/robots/quad/quad_camera.urdf (robot description, URDF)
Before this commit: robot quadrotor, 11 links, 10 joints
Links:
- link downward_camera_link: geometry visual box size=0.1 0.05 0.02
- link rectangular_link: geometry visual box size=0.1 0.05 0.02
